Commit message: Add files via upload

File: mp500lwa4d_description/urdf/lwa4dmp500.urdf.xacro (robot description, xacro)
@@ -5,44 +5,46 @@
   <xacro:property name="M_PI" value="3.1415926535897931" />
   <xacro:property name="safety_offset" value="0.02"/>
+  <xacro:include filename="$(find mp500lwa4d_description)/urdf/materials.urdf.xacro"/>
+  <xacro:include filename="$(find mp500lwa4d_description)/urdf/common.xacro"/>
 <!-- Materials -->
-    <material name="Neobotix/Black">
-        <color rgba="0.0 0.0 0.0 1.0"/>
-    </material>
-    <material name="Neobotix/Blue">
-        <color rgba="0.0 0.0 0.8 1.0"/>
-    </material>
-    <material name="Neobotix/Green">
-        <color rgba="0.0 0.8 0.0 1.0"/>
-    </material>
-    <material name="Neobotix/Grey">
-        <color rgba="0.7 0.7 0.7 1.0"/>
-    </material>
-    <material name="Neobotix/Grey2">
-        <color rgba="0.9 0.9 0.9 1.0"/>
-    </material>
-    <material name="Neobotix/Red">
-        <color rgba="0.8 0.0 0.0 1.0"/>
-    </material>
-    <material name="Neobotix/White">
-        <color rgba="1.0 1.0 1.0 1.0"/>
-    </material>
-    <material name="Neobotix/Yellow">
-        <color rgba="1.0 1.0 0 10" />
-    </material>
-   <material name="Schunk/LightGrey">
-        <color rgba="0.7 0.7 0.7 1.0"/>
-   </material>
-   <material name="Schunk/DarkGrey">
-        <color rgba="0.4 0.4 0.4 1.0"/>
-   </material>
-   <material name="Schunk/Black">
-        <color rgba="0.0 0.0 0.0 1.0"/>
-   </material>
-   <material name="Schunk/DarkGolden">
-        <color rgba="0.4 0.4 0.3 1.0"/>
-   </material>
-   <material name="Schunk/Blue">
-        <color rgba="0.0 0.0 0.8 1.0"/>
-   </material>
+  <!--material name="Neobotix/Black">
+    <color rgba="0.0 0.0 0.0 1.0"/>
+  </material>
+  <material name="Neobotix/Blue">
+    <color rgba="0.0 0.0 0.8 1.0"/>
+  </material>
+  <material name="Neobotix/Green">
+    <color rgba="0.0 0.8 0.0 1.0"/>
+  </material>
+  <material name="Neobotix/Grey">
+    <color rgba="0.7 0.7 0.7 1.0"/>
+  </material>
+  <material name="Neobotix/Grey2">
+    <color rgba="0.9 0.9 0.9 1.0"/>
+  </material>
+  <material name="Neobotix/Red">
+    <color rgba="0.8 0.0 0.0 1.0"/>
+  </material>
+  <material name="Neobotix/White">
+    <color rgba="1.0 1.0 1.0 1.0"/>
+  </material>
+  <material name="Neobotix/Yellow">
+    <color rgba="1.0 1.0 0 10" />
+  </material>
+  <material name="Schunk/LightGrey">
+    <color rgba="0.7 0.7 0.7 1.0"/>
+  </material>
+  <material name="Schunk/DarkGrey">
+    <color rgba="0.4 0.4 0.4 1.0"/>
+  </material>
+  <material name="Schunk/Black">
+    <color rgba="0.0 0.0 0.0 1.0"/>
+  </material>
+  <material name="Schunk/DarkGolden">
+    <color rgba="0.4 0.4 0.3 1.0"/>
+  </material>
+  <material name="Schunk/Blue">
+    <color rgba="0.0 0.0 0.8 1.0"/>
+  </material-->
   <!--neo_mp_500-->
   <!--xacro:include filename="$(find neo_mp_500)/robot_model/mp_500/mp500.urdf.xacro" /-->
@@ -50,244 +52,214 @@
 <!--++++++++++++++++++++body++++++++++++++++++++++++++++-->
   <link name="base_link">
-       <inertial>
-          <mass value="25.67" />
-	    <origin xyz="0 0 0.216" rpy="0 0 0"/>
-	<inertia ixx="0.54" ixy="0.0" ixz="0.0" iyy="1.08" iyz="0.0" izz="1.23" />
-       </inertial>
-       <visual name='body'>
-        <!--origin xyz="0.0 0.0 0.234" rpy="0 0 1.57" /--><!-- for cylinder -->
-	<origin xyz="-0.160 0.0 0.09" rpy="0 0 -1.57" /><!-- for STL -->
-              <geometry>
-                 <mesh filename="package://neo_mp_500/robot_model/mp_500/meshes/MP500-BODY.STL" scale="0.01 0.01 0.01"/>
-	    	<!--cylinder length="0.381" radius="0.2545"/-->
-	    	<!--box size="0.445 0.277 0.17"/-->
-              </geometry>
-        <material name="Neobotix/Grey" />
-       </visual>
-      <collision name='body_collision'>
-        <origin xyz="0 0 0.216" rpy="0 0 -1.57" />
-        <geometry>
-          <box size="0.400 0.676 0.300"/>
-          <!--cylinder length="0.381" radius="0.2545"/-->
-        </geometry>
-      </collision>
-   </link>
+    <inertial>
+      <mass value="25.67" />
+      <origin xyz="0 0 0.216" rpy="0 0 0"/>
+      <inertia ixx="0.54" ixy="0.0" ixz="0.0" iyy="1.08" iyz="0.0" izz="1.23" />
+    </inertial>
+    <visual name='body'>
+      <!--origin xyz="0.0 0.0 0.234" rpy="0 0 1.57" /--><!-- for cylinder -->
+      <origin xyz="-0.160 0.0 0.09" rpy="0 0 -1.57" /><!-- for STL -->
+      <geometry>
+        <mesh filename="package://neo_mp_500/robot_model/mp_500/meshes/MP500-BODY.STL" scale="0.01 0.01 0.01"/>
+        <!--cylinder length="0.381" radius="0.2545"/-->
+        <!--box size="0.445 0.277 0.17"/-->
+      </geometry>
+      <material name="Neobotix/Grey" />
+    </visual>
+    <collision name='body_collision'>
+      <origin xyz="0 0 0.216" rpy="0 0 -1.57" />
+      <geometry>
+        <box size="0.400 0.676 0.300"/>
+        <!--cylinder length="0.381" radius="0.2545"/-->
+      </geometry>
+    </collision>
+  </link>
 <!--+++++++++++++++++++wheel_left_link++++++++++++++++++++++++-->
-   <link name="wheel_left_link" type="wheel">
-      <inertial>
-      	<mass value="1.0" />
-     	   <origin xyz="0 0 0" rpy="0 0 0" />
-      	 <inertia ixx="0.0045" ixy="0" ixz="0" iyy="0.0078" iyz="0" izz="0.0045" />
-      </inertial>
-      <visual>
-     	<origin xyz="0 0 0" rpy="0 0 -1.57" />
-     	<geometry>
-		<mesh filename="package://neo_mp_500/robot_model/mp_500/meshes/MP500-WHEEL.STL" scale="0.01 0.01 0.01" />
-     	</geometry>
-     	<material name="Neobotix/Black" />
-      </visual>
-    <collision>
-     	<origin xyz="0 0 0" rpy="0 1.57 -1.57" />
-     	<geometry>
-        	<cylinder radius="0.125" length="0.085"/>
-     	</geometry>
-    </collision>
-</link>
+  <link name="wheel_left_link" type="wheel">
+    <inertial>
+      <mass value="1.0" />
+      <origin xyz="0 0 0" rpy="0 0 0" />
+      <inertia ixx="0.0045" ixy="0" ixz="0" iyy="0.0078" iyz="0" izz="0.0045" />
+    </inertial>
+    <visual>
+      <origin xyz="0 0 0" rpy="0 0 -1.57" />
+      <geometry>
+	<mesh filename="package://neo_mp_500/robot_model/mp_500/meshes/MP500-WHEEL.STL" scale="0.01 0.01 0.01" />
+      </geometry>
+      <material name="Neobotix/Black" />
+    </visual>
+    <collision>
+      <origin xyz="0 0 0" rpy="0 1.57 -1.57" />
+      <geometry>
+        <cylinder radius="0.125" length="0.085"/>
+      </geometry>
+    </collision>
+  </link>
 <!--+++++++++++++++++++wheel_left_joint++++++++++++++++++++++++-->
   <joint name="wheel_left_joint" type="revolute">
-     <origin xyz="-0.155 0.255 0.13" rpy="0 0 0" />
-    	<axis xyz="0 1 0"/>
-    	<limit effort="10000.0" lower="-1e+16" upper="1e+16" velocity="11.6"/>
-    	<joint_properties damping="0.0" friction="0.0" />
-    	<parent link="base_link" />
-     <child link="wheel_left_link" />
-    </joint>
+    <origin xyz="-0.155 0.255 0.13" rpy="0 0 0" />
+    <axis xyz="0 1 0"/>
+    <limit effort="10000.0" lower="-1e+16" upper="1e+16" velocity="11.6"/>
+    <joint_properties damping="0.0" friction="0.0" />
+    <parent link="base_link" />
+    <child link="wheel_left_link" />
+  </joint>
 <!--+++++++++++++++++++wheel_right_link++++++++++++++++++++++++-->
-<!--Mesh Volume is 3587.704102
-Mesh Surface is 1876.550415
-Thin shell barycenter -25.340059 -0.000027 4.499997
-Center of Mass is -25.340000 -0.000164 4.500009
-Inertia Tensor is :
-| 322624.937500 -0.068522 -1.293689 |
-| -0.068522 179104.328125 -1.342927 |
-| -1.293689 -1.342927 179079.796875 |
-Principal axes are :
-| 1.000000 -0.000000 0.000009 |
-| -0.000000 0.998514 0.054499 |
-| -0.000009 -0.054499 0.998514 |
-axis momenta are :
-| 322624.937500 179104.406250 179079.718750 |
-Mesh Volume is 0.000000
-Mesh Surface is 0.000019
-Thin shell barycenter -0.002534 -0.000000 0.000450
-Center of Mass is -0.002534 -0.000000 0.000450
-Inertia Tensor is :
-| 0.000000 -0.000000 -0.000000 |
-| -0.000000 0.000000 -0.000000 |
-| -0.000000 -0.000000 0.000000 |
-Principal axes are :
-| 1.000000 -0.000000 0.000009 |
-| -0.000000 0.998526 0.054276 |
-| -0.000009 -0.054276 0.998526 |
-axis momenta are :
-| 0.000000 0.000000 0.000000 | -->
   <link name="wheel_right_link" type="wheel">
-     <inertial>
+    <inertial>
       <mass value="1" />
       <origin xyz="0 0 0" rpy="0 0 0" />
-		  <!--inertia ixx="0.0051" ixy="0" ixz="0" iyy="0.0051" iyz="0" izz="0.009" /-->
-       <inertia ixx="0.0045" ixy="0" ixz="0" iyy="0.0078" iyz="0" izz="0.0045" />
-     </inertial>
-     <visual>
-	<origin xyz="0 0 0" rpy="0 0 -1.57" />
-	<geometry>
-	 <mesh filename="package://neo_mp_500/robot_model/mp_500/meshes/MP500-WHEEL.STL" scale="0.01 0.01 0.01" />
-	</geometry>
-	<material name="Neobotix/Black" />
-     </visual>
-     <collision>
-	<origin xyz="0 0 0" rpy="0 1.57 -1.57" />
-	<geometry>
-		<cylinder radius="0.125" length="0.085"/>
-	</geometry>
-    </collision>
-   </link>
+      <!--inertia ixx="0.0051" ixy="0" ixz="0" iyy="0.0051" iyz="0" izz="0.009" /-->
+      <inertia ixx="0.0045" ixy="0" ixz="0" iyy="0.0078" iyz="0" izz="0.0045" />
+    </inertial>
+    <visual>
+      <origin xyz="0 0 0" rpy="0 0 -1.57" />
+      <geometry>
+	<mesh filename="package://neo_mp_500/robot_model/mp_500/meshes/MP500-WHEEL.STL" scale="0.01 0.01 0.01" />
+      </geometry>
+      <material name="Neobotix/Black"/>
+    </visual>
+    <collision>
+      <origin xyz="0 0 0" rpy="0 1.57 -1.57" />
+      <geometry>
+	<cylinder radius="0.125" length="0.085"/>
+      </geometry>
+    </collision>
+  </link>
 <!--+++++++++++++++++++wheel_right_joint++++++++++++++++++++++++-->
-   <joint name="wheel_right_joint" type="revolute">
-     <origin xyz="-0.155 -0.255 0.13" rpy="0 0 0" />
-    	<axis xyz="0 1 0"/>
-    	<limit effort="10000.0" lower="-1e+16" upper="1e+16" velocity="11.6"/>
-    	<joint_properties damping="0.0" friction="0.0" />
-    	<parent link="base_link" />
-    	<child link="wheel_right_link" />
-    </joint>
+  <joint name="wheel_right_joint" type="revolute">
+    <origin xyz="-0.155 -0.255 0.13" rpy="0 0 0" />
+    <axis xyz="0 1 0"/>
+    <limit effort="10000.0" lower="-1e+16" upper="1e+16" velocity="11.6"/>
+    <joint_properties damping="0.0" friction="0.0" />
+    <parent link="base_link" />
+    <child link="wheel_right_link" />
+  </joint>
 <!--+++++++++++++++++++laserscanner_front_joint++++++++++++++++++++++++-->
-   <joint name="laserscanner_front_joint" type="fixed">
-     <axis xyz="0 0 1" />
-     <origin xyz="-0.39 0 0.281" rpy="0 0 0" />
-     <parent link="base_link"/>
-     <child link="laserscanner_front_link"/>
-   </joint>
+  <joint name="laserscanner_front_joint" type="fixed">
+    <axis xyz="0 0 1" />
+    <origin xyz="-0.39 0 0.281" rpy="0 0 0" />
+    <parent link="base_link"/>
+    <child link="laserscanner_front_link"/>
+  </joint>
 <!--+++++++++++++++++++laserscanner_front_link++++++++++++++++++++++++-->
-   <link name="laserscanner_front_link" type="laser">
-	<inertial>
-		<mass value="0.01" />
-		<origin xyz="0 0 0" rpy="3.14 0 -1.57" />
-		<inertia ixx="0.001" ixy="0" ixz="0" iyy="0.001" iyz="0" izz="0.001" />
-        </inertial>
- 	<visual>
-		<origin xyz="0 0 -0.04" rpy="3.14 0 -1.57" />
-		<geometry>
-                            <!--cylinder length="0.154" radius="0.053" /-->
-                     <mesh filename="package://neo_mp_500/robot_model/mp_500/meshes/SICK-S300.STL" />
-		</geometry>
-		<material name="Neobotix/Yellow" />
-  	</visual>
-  	<collision>
-		<origin xyz="0 0 0" rpy="3.14 0 -1.57" />
-		<geometry>
-	  	<cylinder length="0.154" radius="0.053" />
-		</geometry>
-  	</collision>
-   </link>
+  <link name="laserscanner_front_link" type="laser">
+    <inertial>
+      <mass value="0.01" />
+      <origin xyz="0 0 0" rpy="3.14 0 -1.57" />
+      <inertia ixx="0.001" ixy="0" ixz="0" iyy="0.001" iyz="0" izz="0.001" />
+    </inertial>
+    <visual>
+      <origin xyz="0 0 -0.04" rpy="3.14 0 -1.57" />
+      <geometry>
+        <!--cylinder length="0.154" radius="0.053" /-->
+        <mesh filename="package://neo_mp_500/robot_model/mp_500/meshes/SICK-S300.STL" />
+      </geometry>
+      <material name="Neobotix/Yellow"/>
+    </visual>
+    <collision>
+      <origin xyz="0 0 0" rpy="3.14 0 -1.57" />
+      <geometry>
+	<cylinder length="0.154" radius="0.053" />
+      </geometry>
+    </collision>
+  </link>
 <!--+++++++++++++++ wheel_hanger+++++++++++++++++++++++++++-->
-   <link name="hanger">
-      <inertial>
-		  <mass value="0.01" />
-		  <origin xyz="0 0 0" rpy="0 0 0" />
-		  <inertia ixx="0.0013" ixy="0" ixz="0" iyy="0.0013" iyz="0" izz="0.0013" />
-      </inertial>
-      <visual>
-	<origin xyz="0 0 0" rpy="0 0 -1.57" />
-	<geometry>
-	      <mesh filename="package://neo_mp_500/robot_model/mp_500/meshes/HANGER-WHEEL.STL" scale="0.01 0.01 0.01" />
-	 </geometry>
-	 <material name="Neobotix/Grey" />
-	</visual>
-       <collision>
-		 <origin xyz="0 0 0" rpy="0 0 -1.57" />
-		 <geometry>
-          	 <sphere radius="0.00115"/>
-		 </geometry>
-       </collision>
-   </link>
-   <joint name="hanger_joint" type="fixed">
-    	<origin xyz="0.255 0 0.11" rpy="0 0 0"/>
-    	<axis xyz="0 0 1"/>
-    	<limit effort="10000.0" lower="-1e+16" upper="1e+16" velocity="13.5"/>
-    	<joint_properties damping="0.0" friction="0.0" />
-    	<parent link="base_link" />
-    	<child link="hanger" />
-   </joint>
+  <link name="hanger">
+    <inertial>
+      <mass value="0.01" />
+      <origin xyz="0 0 0" rpy="0 0 0" />
+      <inertia ixx="0.0013" ixy="0" ixz="0" iyy="0.0013" iyz="0" izz="0.0013" />
+    </inertial>
+    <visual>
+      <origin xyz="0 0 0" rpy="0 0 -1.57" />
+      <geometry>
+	<mesh filename="package://neo_mp_500/robot_model/mp_500/meshes/HANGER-WHEEL.STL" scale="0.01 0.01 0.01" />
+      </geometry>
+      <material name="Neobotix/Grey"/>
+    </visual>
+    <collision>
+      <origin xyz="0 0 0" rpy="0 0 -1.57" />
+      <geometry>
+        <sphere radius="0.00115"/>
+      </geometry>
+    </collision>
+  </link>
+  <joint name="hanger_joint" type="fixed">
+    <origin xyz="0.255 0 0.11" rpy="0 0 0"/>
+    <axis xyz="0 0 1"/>
+    <limit effort="10000.0" lower="-1e+16" upper="1e+16" velocity="13.5"/>
+    <joint_properties damping="0.0" friction="0.0" />
+    <parent link="base_link" />
+    <child link="hanger" />
+  </joint>
 <!--+++++++++++++++ castor_front +++++++++++++++++++++++++++-->
-   <link name="castor_front">
-	<inertial>
-	  <mass value="0.25" />
-	  <origin xyz="0 0 0" rpy="0 0 0" />
-	  <inertia ixx="0.000025" ixy="0" ixz="0" iyy="0.000025" iyz="0" izz="0.000025" />
-	</inertial>
-	<visual>
-	  <origin xyz="0 0 0" rpy="0 0 0" />
-	  <geometry>
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
Commit message: Add files via upload

File: mp500lwa4d_description/urdf/lwa4dmp500.urdf.xacro (robot description, xacro)
@@ -80,5 +80,5 @@
       <mass value="1.0" />
       <origin xyz="0 0 0" rpy="0 0 0" />
-      <inertia ixx="0.0045" ixy="0" ixz="0" iyy="0.0078" iyz="0" izz="0.0045" />
+      <inertia ixx="0.0045" ixy="0" ixz="0" iyy="0.0078125" iyz="0" izz="0.0045" />
     </inertial>
     <visual>
@@ -111,5 +111,5 @@
       <origin xyz="0 0 0" rpy="0 0 0" />
       <!--inertia ixx="0.0051" ixy="0" ixz="0" iyy="0.0051" iyz="0" izz="0.009" /-->
-      <inertia ixx="0.0045" ixy="0" ixz="0" iyy="0.0078" iyz="0" izz="0.0045" />
+      <inertia ixx="0.0045" ixy="0" ixz="0" iyy="0.0078125" iyz="0" izz="0.0045" />
     </inertial>
     <visual>
@@ -148,5 +148,5 @@
       <mass value="0.01" />
       <origin xyz="0 0 0" rpy="3.14 0 -1.57" />
-      <inertia ixx="0.001" ixy="0" ixz="0" iyy="0.001" iyz="0" izz="0.001" />
+      <inertia ixx="0.0001" ixy="0" ixz="0" iyy="0.0001" iyz="0" izz="0.0001" />
     </inertial>
     <visual>
@@ -170,5 +170,5 @@
       <mass value="0.01" />
       <origin xyz="0 0 0" rpy="0 0 0" />
-      <inertia ixx="0.0013" ixy="0" ixz="0" iyy="0.0013" iyz="0" izz="0.0013" />
+      <inertia ixx="0.00013" ixy="0" ixz="0" iyy="0.00013" iyz="0" izz="0.00013" />
     </inertial>
     <visual>
@@ -222,5 +222,5 @@
   </gazebo>
   <joint name="castor_front_joint" type="fixed">
-    <origin xyz="0.48 0 0.01" rpy="0 0 0"/>
+    <origin xyz="0.32 0 0.01" rpy="0 0 0"/>
      <!--limit effort="100.0" velocity="13.5"/>
     <joint_properties damping="0.0" friction="0.0" /-->
@@ -229,5 +229,5 @@
   </joint>
 <!--+++++++++++++++ castor_back +++++++++++++++++++++++++++-->
-  <link name="castor_back">
+  <!--link name="castor_back">
     <inertial>
     <mass value="0.25" />
@@ -254,12 +254,10 @@
    <kp  value="1.0" />
    <kd  value="1.0" />
-  </gazebo>
-  <joint name="castor_back_joint" type="fixed">
-    <origin xyz="-0.35 0 0.01" rpy="0 0 0"/>
-    <!--limit effort="100.0" velocity="13.5"/>
-    <joint_properties damping="0.0" friction="0.0" /-->
+  </gazebo-->
+  <!--joint name="castor_back_joint" type="fixed">
+    <origin xyz="-0.30 0 0.01" rpy="0 0 0"/>
     <parent link="base_link" />
     <child link="castor_back" />
-  </joint>
+  </joint-->
   <!--xacro:include filename="$(find schunk_description)/urdf/common.xacro" /-->
   <!--xacro:include filename="$(find schunk_description)/urdf/materials.urdf.xacro" /-->
@@ -277,7 +275,7 @@
   <link name="arm_podest_link">
     <inertial>
-      <mass value="0.01" />
-      <origin xyz="0 0 0" />
-      <inertia ixx="0.001" ixy="0.0" ixz="0.0" iyy="0.001" iyz="0.0" izz="0.001" />
+      <mass value="2" />
+      <origin xyz="0 0 0" />
+      <inertia ixx="0.01" ixy="0.0" ixz="0.0" iyy="0.01" iyz="0.0" izz="0.01" />
     </inertial>
     <visual>
@@ -302,7 +300,7 @@
     <!--xacro:default_inertial/-->
     <inertial>
-      <mass value="0.01" />
-      <origin xyz="0 0 0" />
-      <inertia ixx="0.001" ixy="0.0" ixz="0.0" iyy="0.001" iyz="0.0" izz="0.001" />
+      <mass value="2" />
+      <origin xyz="0 0 0" />
+      <inertia ixx="0.01" ixy="0.0" ixz="0.0" iyy="0.01" iyz="0.0" izz="0.01" />
     </inertial>
   </link>
@@ -318,7 +316,7 @@
   <link name="arm_1_link">
     <inertial>
-      <mass value="0.01" />
-      <origin xyz="0 0 0" />
-      <inertia ixx="0.001" ixy="0.0" ixz="0.0" iyy="0.001" iyz="0.0" izz="0.001" />
+      <mass value="2" />
+      <origin xyz="0 0 0" />
+      <inertia ixx="0.01" ixy="0.0" ixz="0.0" iyy="0.01" iyz="0.0" izz="0.01" />
     </inertial>
     <visual>
@@ -345,7 +343,7 @@
   <link name="arm_2_link">
     <inertial>
-      <mass value="0.01" />
-      <origin xyz="0 0 0" />
-      <inertia ixx="0.001" ixy="0.0" ixz="0.0" iyy="0.001" iyz="0.0" izz="0.001" />
+      <mass value="2" />
+      <origin xyz="0 0 0" />
+      <inertia ixx="0.01" ixy="0.0" ixz="0.0" iyy="0.01" iyz="0.0" izz="0.01" />
     </inertial>
     <visual>
@@ -372,7 +370,7 @@
   <link name="arm_3_link">
     <inertial>
-      <mass value="0.01" />
-      <origin xyz="0 0 0" />
-      <inertia ixx="0.001" ixy="0.0" ixz="0.0" iyy="0.001" iyz="0.0" izz="0.001" />
+      <mass value="2" />
+      <origin xyz="0 0 0" />
+      <inertia ixx="0.01" ixy="0.0" ixz="0.0" iyy="0.01" iyz="0.0" izz="0.01" />
     </inertial>
     <visual>
@@ -399,7 +397,7 @@
   <link name="arm_4_link">
     <inertial>
-      <mass value="0.01" />
-      <origin xyz="0 0 0" />
-      <inertia ixx="0.001" ixy="0.0" ixz="0.0" iyy="0.001" iyz="0.0" izz="0.001" />
+      <mass value="2" />
+      <origin xyz="0 0 0" />
+      <inertia ixx="0.01" ixy="0.0" ixz="0.0" iyy="0.01" iyz="0.0" izz="0.01" />
     </inertial>
     <visual>
@@ -426,7 +424,7 @@
   <link name="arm_5_link">
     <inertial>
-      <mass value="0.01" />
-      <origin xyz="0 0 0" />
-      <inertia ixx="0.001" ixy="0.0" ixz="0.0" iyy="0.001" iyz="0.0" izz="0.001" />
+      <mass value="2" />
+      <origin xyz="0 0 0" />
+      <inertia ixx="0.01" ixy="0.0" ixz="0.0" iyy="0.01" iyz="0.0" izz="0.01" />
     </inertial>
     <visual>
@@ -453,7 +451,7 @@
   <link name="arm_6_link">
     <inertial>
-      <mass value="0.01" />
-      <origin xyz="0 0 0" />
-      <inertia ixx="0.001" ixy="0.0" ixz="0.0" iyy="0.001" iyz="0.0" izz="0.001" />
+      <mass value="2" />
+      <origin xyz="0 0 0" />
+      <inertia ixx="0.01" ixy="0.0" ixz="0.0" iyy="0.01" iyz="0.0" izz="0.01" />
     </inertial>
     <visual>
@@ -480,7 +478,7 @@
   <link name="arm_7_link">
     <inertial>
-      <mass value="0.01" />
-      <origin xyz="0 0 0" />
-      <inertia ixx="0.001" ixy="0.0" ixz="0.0" iyy="0.001" iyz="0.0" izz="0.001" />
+      <mass value="2" />
+      <origin xyz="0 0 0" />
+      <inertia ixx="0.01" ixy="0.0" ixz="0.0" iyy="0.01" iyz="0.0" izz="0.01" />
     </inertial>
     <visual>
@@ -504,7 +502,7 @@
   <link name="arm_ee_link">
     <inertial>
-      <mass value="0.01" />
-      <origin xyz="0 0 0" />
-      <inertia ixx="0.001" ixy="0.0" ixz="0.0" iyy="0.001" iyz="0.0" izz="0.001" />
+      <mass value="1" />
+      <origin xyz="0 0 0" />
+      <inertia ixx="0.005" ixy="0.0" ixz="0.0" iyy="0.005" iyz="0.0" izz="0.005" />
     </inertial>
   </link>
@@ -662,13 +660,8 @@
     <odometrySource>encoder</odometrySource>
   </plugin>
-  <!--plugin name="ros_control" filename="libhwi_switch_gazebo_ros_control.so"-->
-  <plugin name="gazebo_ros_control" filename="libgazebo_ros_control.so">
-    <!--plugin name="ros_control" filename="libhwi_switch_gazebo_ros_control.so"-->
+    <plugin name="gazebo_ros_control" filename="libgazebo_ros_control.so">
     <robotNamespace>mp500lwa4d</robotNamespace>
     <filterJointsParam>joint_names</filterJointsParam>
   </plugin>
-  <!--plugin name="joint_state_publisher" filename="libgazebo_ros_joint_state_publisher.so">
-  <jointName>wheel_left_joint, wheel_right_joint</jointName>
-  </plugin>>-->
 </gazebo>
 </robot>
