Commit message: Add files via upload

File: mp500lwa4d_description/urdf/lwa4dmp500.urdf.xacro (robot description, xacro)
@@ -213,5 +213,5 @@
       <mass value="2" />
       <origin xyz="0 0 0" />
-      <inertia ixx="0.01" ixy="0.0" ixz="0.0" iyy="0.01" iyz="0.0" izz="0.01" />
+      <inertia ixx="0.0091" ixy="0.0" ixz="0.0" iyy="0.0091" iyz="0.0" izz="0.0049" />
     </inertial>
     <visual>
@@ -236,7 +236,7 @@
     <!--xacro:default_inertial/-->
     <inertial>
-      <mass value="2" />
-      <origin xyz="0 0 0" />
-      <inertia ixx="0.01" ixy="0.0" ixz="0.0" iyy="0.01" iyz="0.0" izz="0.01" />
+      <mass value="0.02" />
+      <origin xyz="0 0 0" />
+      <inertia ixx="0.00001" ixy="0.0" ixz="0.0" iyy="0.00001" iyz="0.0" izz="0.00001" />
     </inertial>
   </link>
@@ -254,5 +254,5 @@
       <mass value="2" />
       <origin xyz="0 0 0" />
-      <inertia ixx="0.01" ixy="0.0" ixz="0.0" iyy="0.01" iyz="0.0" izz="0.01" />
+      <inertia ixx="0.0091" ixy="0.0" ixz="0.0" iyy="0.0091" iyz="0.0" izz="0.005" />
     </inertial>
     <visual>
@@ -281,5 +281,5 @@
       <mass value="2" />
       <origin xyz="0 0 0" />
-      <inertia ixx="0.01" ixy="0.0" ixz="0.0" iyy="0.01" iyz="0.0" izz="0.01" />
+      <inertia ixx="0.0091" ixy="0.0" ixz="0.0" iyy="0.0049" iyz="0.0" izz="0.0091" />
     </inertial>
     <visual>
@@ -308,5 +308,5 @@
       <mass value="2" />
       <origin xyz="0 0 0" />
-      <inertia ixx="0.01" ixy="0.0" ixz="0.0" iyy="0.01" iyz="0.0" izz="0.01" />
+      <inertia ixx="0.0091" ixy="0.0" ixz="0.0" iyy="0.0091" iyz="0.0" izz="0.0049" />
     </inertial>
     <visual>
@@ -335,5 +335,5 @@
       <mass value="2" />
       <origin xyz="0 0 0" />
-      <inertia ixx="0.01" ixy="0.0" ixz="0.0" iyy="0.01" iyz="0.0" izz="0.01" />
+      <inertia ixx="0.0091" ixy="0.0" ixz="0.0" iyy="0.0049" iyz="0.0" izz="0.0091" />
     </inertial>
     <visual>
@@ -362,5 +362,5 @@
       <mass value="2" />
       <origin xyz="0 0 0" />
-      <inertia ixx="0.01" ixy="0.0" ixz="0.0" iyy="0.01" iyz="0.0" izz="0.01" />
+      <inertia ixx="0.0091" ixy="0.0" ixz="0.0" iyy="0.0049" iyz="0.0" izz="0.0091" />
     </inertial>
     <visual>
@@ -387,7 +387,7 @@
   <link name="arm_6_link">
     <inertial>
-      <mass value="2" />
-      <origin xyz="0 0 0" />
-      <inertia ixx="0.01" ixy="0.0" ixz="0.0" iyy="0.01" iyz="0.0" izz="0.01" />
+      <mass value="1" />
+      <origin xyz="0 0 0" />
+      <inertia ixx="0.00196" ixy="0.0" ixz="0.0" iyy="0.00196" iyz="0.0" izz="0.00196" />
     </inertial>
     <visual>
@@ -414,7 +414,7 @@
   <link name="arm_7_link">
     <inertial>
-      <mass value="2" />
-      <origin xyz="0 0 0" />
-      <inertia ixx="0.01" ixy="0.0" ixz="0.0" iyy="0.01" iyz="0.0" izz="0.01" />
+      <mass value="0.5" />
+      <origin xyz="0 0 0" />
+      <inertia ixx="0.001" ixy="0.0" ixz="0.0" iyy="0.001" iyz="0.0" izz="0.001" />
     </inertial>
     <visual>
@@ -438,7 +438,7 @@
   <link name="arm_ee_link">
     <inertial>
-      <mass value="1" />
-      <origin xyz="0 0 0" />
-      <inertia ixx="0.005" ixy="0.0" ixz="0.0" iyy="0.005" iyz="0.0" izz="0.005" />
+      <mass value="0.01" />
+      <origin xyz="0 0 0" />
+      <inertia ixx="0.00005" ixy="0.0" ixz="0.0" iyy="0.00005" iyz="0.0" izz="0.00005" />
     </inertial>
   </link>

Commit message: Add files via upload

File: mp500lwa4d_description/urdf/lwa4dmp500.urdf.xacro (robot description, xacro)
@@ -7,9 +7,5 @@
   <xacro:include filename="$(find mp500lwa4d_description)/urdf/materials.urdf.xacro"/>
   <xacro:include filename="$(find mp500lwa4d_description)/urdf/common.xacro"/>
-<!-- Materials -->
-  <!--neo_mp_500-->
-  <!--xacro:include filename="$(find neo_mp_500)/robot_model/mp_500/mp500.urdf.xacro" /-->
 <!--++++++++++++++++++++++++++++++base_link++++++++++++++++++++++++++++++++++++++++++++++++++++-->
-<!--++++++++++++++++++++body++++++++++++++++++++++++++++-->
   <link name="base_link">
     <inertial>
@@ -35,4 +31,23 @@
       </geometry>
     </collision>
+    <visual name="castor_front">
+      <origin xyz="0.32 0 0.01" rpy="0 0 0" />
+      <geometry>
+        <sphere radius="0.005"/>
+      </geometry>
+      <material name="Neobotix/Grey"/>
+    </visual>
+    <collision>
+      <origin xyz="0.32 0 0.01" rpy="0 0 0" />
+      <geometry>
+        <sphere radius="0.005"/>
+      </geometry>
+    </collision>
+  <!--gazebo reference="caster_front">
+    <mu1 value="0" />
+    <mu2 value="0" />
+    <kp  value="1.0" />
+    <kd  value="1.0" />
+  </gazebo-->
   </link>
   <link name="mobile_dummy_link">
@@ -133,74 +148,4 @@
     </collision>
   </link>
-<!--+++++++++++++++ wheel_hanger+++++++++++++++++++++++++++-->
-  <link name="hanger">
-    <inertial>
-      <mass value="0.01" />
-      <origin xyz="0 0 0" rpy="0 0 0" />
-      <inertia ixx="0.00013" ixy="0" ixz="0" iyy="0.00013" iyz="0" izz="0.00013" />
-    </inertial>
-    <visual>
-      <origin xyz="0 0 0" rpy="0 0 -1.57" />
-      <geometry>
-	<mesh filename="package://mp500lwa4d_description/meshes/HANGER-WHEEL.STL" scale="0.01 0.01 0.01" />
-      </geometry>
-      <material name="Neobotix/Grey"/>
-    </visual>
-    <collision>
-      <origin xyz="0 0 0" rpy="0 0 -1.57" />
-      <geometry>
-        <sphere radius="0.00115"/>
-      </geometry>
-    </collision>
-  </link>
-  <joint name="hanger_joint" type="fixed">
-    <origin xyz="0.255 0 0.11" rpy="0 0 0"/>
-    <axis xyz="0 0 1"/>
-    <limit effort="1000.0" lower="-1e+16" upper="1e+16" velocity="13.5"/>
-    <joint_properties damping="0.0" friction="0.0" />
-    <parent link="base_link" />
-    <child link="hanger" />
-  </joint>
-<!--+++++++++++++++ castor_front +++++++++++++++++++++++++++-->
-  <link name="castor_front">
-    <!--inertial>
-      <mass value="0.25" />
-      <origin xyz="0 0 0" rpy="0 0 0" />
-      <inertia ixx="0.000025" ixy="0" ixz="0" iyy="0.000025" iyz="0" izz="0.000025" />
-    </inertial-->
-    <visual>
-      <origin xyz="0 0 0" rpy="0 0 0" />
-      <geometry>
-        <sphere radius="0.005"/>
-      </geometry>
-      <material name="Neobotix/Grey"/>
-    </visual>
-    <collision>
-      <origin xyz="0 0 0" rpy="0 0 0" />
-      <geometry>
-        <sphere radius="0.005"/>
-      </geometry>
-    </collision>
-  </link>
-  <gazebo reference="caster_front">
-    <mu1 value="0" />
-    <mu2 value="0" />
-    <kp  value="1.0" />
-    <kd  value="1.0" />
-  </gazebo>
-  <joint name="castor_front_joint" type="fixed">
-    <origin xyz="0.32 0 0.01" rpy="0 0 0"/>
-     <!--limit effort="100.0" velocity="13.5"/>
-    <joint_properties damping="0.0" friction="0.0" /-->
-    <parent link="base_link" />
-    <child link="castor_front" />
-  </joint>
-  <!--xacro:include filename="$(find schunk_description)/urdf/common.xacro" /-->
-  <!--xacro:include filename="$(find schunk_description)/urdf/materials.urdf.xacro" /-->
-  <!-- schunk lwa4d -->
-  <!--xacro:include filename="$(find schunk_description)/urdf/lwa4d/lwa4d.urdf.xacro" /-->
-  <!--xacro:include filename="$(find schunk_description)/urdf/common.xacro" /-->
-  <!--xacro:include filename="$(find schunk_description)/urdf/lwa4d/lwa4d.gazebo.xacro"/-->
-  <!--xacro:include filename="$(find schunk_description)/urdf/lwa4d/lwa4d.transmission.xacro"/-->
   <!-- joint between base_link and lwa4p_extended_connector_link -->
   <joint name="arm_podest_joint" type="fixed">
