Commit message: Add files via upload

File: mp500lwa4d_description/urdf/common.xacro (robot description, xacro)
@@ -5,4 +5,9 @@
     <self_collide>false</self_collide>
     <material value="Gazebo/Blue"/>
+  </gazebo>
+  <gazebo reference="laserscanner_front_link">
+    <gravity>false</gravity>
+    <self_collide>false</self_collide>
+    <material value="Gazebo/Yellow"/>
   </gazebo>
   <gazebo reference="wheel_right_link">
@@ -69,5 +74,5 @@
     <actuator name="wheel_right_motor">
       <hardwareInterface>hardware_interface/EffortJointInterface</hardwareInterface>
-      <mechanicalReduction>1</mechanicalReduction>
+      <mechanicalReduction>12</mechanicalReduction>
     </actuator>
   </transmission>
@@ -80,5 +85,5 @@
     <actuator name="wheel_left_motor">
       <hardwareInterface>hardware_interface/EffortJointInterface</hardwareInterface>
-      <mechanicalReduction>1</mechanicalReduction>
+      <mechanicalReduction>12</mechanicalReduction>
     </actuator>
   </transmission>
@@ -91,5 +96,5 @@
     </joint>
     <actuator name="arm_1_motor">
-      <mechanicalReduction>1</mechanicalReduction>
+      <mechanicalReduction>596</mechanicalReduction>
     </actuator>
   </transmission>
@@ -102,5 +107,5 @@
     </joint>
     <actuator name="arm_2_motor">
-      <mechanicalReduction>1</mechanicalReduction>
+      <mechanicalReduction>596</mechanicalReduction>
     </actuator>
   </transmission>
@@ -113,5 +118,5 @@
     </joint>
     <actuator name="arm_3_motor">
-      <mechanicalReduction>1</mechanicalReduction>
+      <mechanicalReduction>625</mechanicalReduction>
     </actuator>
   </transmission>
@@ -124,5 +129,5 @@
     </joint>
     <actuator name="arm_4_motor">
-      <mechanicalReduction>1</mechanicalReduction>
+      <mechanicalReduction>625</mechanicalReduction>
     </actuator>
   </transmission>
@@ -135,5 +140,5 @@
     </joint>
     <actuator name="arm_5_motor">
-      <mechanicalReduction>1</mechanicalReduction>
+      <mechanicalReduction>552</mechanicalReduction>
     </actuator>
   </transmission>
@@ -146,5 +151,5 @@
     </joint>
     <actuator name="arm_6_motor">
-      <mechanicalReduction>1</mechanicalReduction>
+      <mechanicalReduction>552</mechanicalReduction>
     </actuator>
   </transmission>
@@ -157,5 +162,5 @@
     </joint>
     <actuator name="arm_7_motor">
-      <mechanicalReduction>1</mechanicalReduction>
+      <mechanicalReduction>300</mechanicalReduction>
     </actuator>
   </transmission>

File: mp500lwa4d_description/urdf/lwa4dmp500.urdf.xacro (robot description, xacro)
@@ -75,4 +75,11 @@
     </collision>
   </link>
+  <link name="mobile_dummy_link">
+  </link>
+  <joint name="mobile_dummy_joint" type="fixed">
+    <parent link="base_link"/>
+    <child link="mobile_dummy_link"/>
+    <origin xyz="0 0 0"/>
+  </joint>
 <!--+++++++++++++++++++wheel_left_link++++++++++++++++++++++++-->
   <link name="wheel_left_link" type="wheel">
@@ -80,5 +87,5 @@
       <mass value="1.0" />
       <origin xyz="0 0 0" rpy="0 0 0" />
-      <inertia ixx="0.0045" ixy="0" ixz="0" iyy="0.0078" iyz="0" izz="0.0045" />
+      <inertia ixx="0.0045" ixy="0" ixz="0" iyy="0.0078125" iyz="0" izz="0.0045" />
     </inertial>
     <visual>
@@ -100,5 +107,5 @@
     <origin xyz="-0.155 0.255 0.13" rpy="0 0 0" />
     <axis xyz="0 1 0"/>
-    <limit effort="10000.0" lower="-1e+16" upper="1e+16" velocity="11.6"/>
+    <limit effort="1000.0" lower="-1e+16" upper="1e+16" velocity="5"/>
     <joint_properties damping="0.0" friction="0.0" />
     <parent link="base_link" />
@@ -111,5 +118,5 @@
       <origin xyz="0 0 0" rpy="0 0 0" />
       <!--inertia ixx="0.0051" ixy="0" ixz="0" iyy="0.0051" iyz="0" izz="0.009" /-->
-      <inertia ixx="0.0045" ixy="0" ixz="0" iyy="0.0078" iyz="0" izz="0.0045" />
+      <inertia ixx="0.0045" ixy="0" ixz="0" iyy="0.0078125" iyz="0" izz="0.0045" />
     </inertial>
     <visual>
@@ -131,5 +138,5 @@
     <origin xyz="-0.155 -0.255 0.13" rpy="0 0 0" />
     <axis xyz="0 1 0"/>
-    <limit effort="10000.0" lower="-1e+16" upper="1e+16" velocity="11.6"/>
+    <limit effort="1000.0" lower="-1e+16" upper="1e+16" velocity="5"/>
     <joint_properties damping="0.0" friction="0.0" />
     <parent link="base_link" />
@@ -148,5 +155,5 @@
       <mass value="0.01" />
       <origin xyz="0 0 0" rpy="3.14 0 -1.57" />
-      <inertia ixx="0.001" ixy="0" ixz="0" iyy="0.001" iyz="0" izz="0.001" />
+      <inertia ixx="0.0001" ixy="0" ixz="0" iyy="0.0001" iyz="0" izz="0.0001" />
     </inertial>
     <visual>
@@ -170,5 +177,5 @@
       <mass value="0.01" />
       <origin xyz="0 0 0" rpy="0 0 0" />
-      <inertia ixx="0.0013" ixy="0" ixz="0" iyy="0.0013" iyz="0" izz="0.0013" />
+      <inertia ixx="0.00013" ixy="0" ixz="0" iyy="0.00013" iyz="0" izz="0.00013" />
     </inertial>
     <visual>
@@ -189,5 +196,5 @@
     <origin xyz="0.255 0 0.11" rpy="0 0 0"/>
     <axis xyz="0 0 1"/>
-    <limit effort="10000.0" lower="-1e+16" upper="1e+16" velocity="13.5"/>
+    <limit effort="1000.0" lower="-1e+16" upper="1e+16" velocity="13.5"/>
     <joint_properties damping="0.0" friction="0.0" />
     <parent link="base_link" />
@@ -196,9 +203,9 @@
 <!--+++++++++++++++ castor_front +++++++++++++++++++++++++++-->
   <link name="castor_front">
-    <inertial>
+    <!--inertial>
       <mass value="0.25" />
       <origin xyz="0 0 0" rpy="0 0 0" />
       <inertia ixx="0.000025" ixy="0" ixz="0" iyy="0.000025" iyz="0" izz="0.000025" />
-    </inertial>
+    </inertial-->
     <visual>
       <origin xyz="0 0 0" rpy="0 0 0" />
@@ -222,5 +229,5 @@
   </gazebo>
   <joint name="castor_front_joint" type="fixed">
-    <origin xyz="0.48 0 0.01" rpy="0 0 0"/>
+    <origin xyz="0.32 0 0.01" rpy="0 0 0"/>
      <!--limit effort="100.0" velocity="13.5"/>
     <joint_properties damping="0.0" friction="0.0" /-->
@@ -229,5 +236,5 @@
   </joint>
 <!--+++++++++++++++ castor_back +++++++++++++++++++++++++++-->
-  <link name="castor_back">
+  <!--link name="castor_back">
     <inertial>
     <mass value="0.25" />
@@ -254,12 +261,10 @@
    <kp  value="1.0" />
    <kd  value="1.0" />
-  </gazebo>
-  <joint name="castor_back_joint" type="fixed">
-    <origin xyz="-0.35 0 0.01" rpy="0 0 0"/>
-    <!--limit effort="100.0" velocity="13.5"/>
-    <joint_properties damping="0.0" friction="0.0" /-->
+  </gazebo-->
+  <!--joint name="castor_back_joint" type="fixed">
+    <origin xyz="-0.30 0 0.01" rpy="0 0 0"/>
     <parent link="base_link" />
     <child link="castor_back" />
-  </joint>
+  </joint-->
   <!--xacro:include filename="$(find schunk_description)/urdf/common.xacro" /-->
   <!--xacro:include filename="$(find schunk_description)/urdf/materials.urdf.xacro" /-->
@@ -277,7 +282,7 @@
   <link name="arm_podest_link">
     <inertial>
-      <mass value="0.01" />
-      <origin xyz="0 0 0" />
-      <inertia ixx="0.001" ixy="0.0" ixz="0.0" iyy="0.001" iyz="0.0" izz="0.001" />
+      <mass value="2" />
+      <origin xyz="0 0 0" />
+      <inertia ixx="0.01" ixy="0.0" ixz="0.0" iyy="0.01" iyz="0.0" izz="0.01" />
     </inertial>
     <visual>
@@ -302,7 +307,7 @@
     <!--xacro:default_inertial/-->
     <inertial>
-      <mass value="0.01" />
-      <origin xyz="0 0 0" />
-      <inertia ixx="0.001" ixy="0.0" ixz="0.0" iyy="0.001" iyz="0.0" izz="0.001" />
+      <mass value="2" />
+      <origin xyz="0 0 0" />
+      <inertia ixx="0.01" ixy="0.0" ixz="0.0" iyy="0.01" iyz="0.0" izz="0.01" />
     </inertial>
   </link>
@@ -313,12 +318,12 @@
     <parent link="arm_base_link"/>
     <child link="arm_1_link"/>
-    <limit effort="216" velocity="0.43633" lower="${-M_PI+safety_offset}" upper="${M_PI-safety_offset}"/>
+    <limit effort="216" velocity="0.4363" lower="${-M_PI+safety_offset}" upper="${M_PI-safety_offset}"/>
   </joint>
 <!-- arm_1_link-->
   <link name="arm_1_link">
     <inertial>
-      <mass value="0.01" />
-      <origin xyz="0 0 0" />
-      <inertia ixx="0.001" ixy="0.0" ixz="0.0" iyy="0.001" iyz="0.0" izz="0.001" />
+      <mass value="2" />
+      <origin xyz="0 0 0" />
+      <inertia ixx="0.01" ixy="0.0" ixz="0.0" iyy="0.01" iyz="0.0" izz="0.01" />
     </inertial>
     <visual>
@@ -345,7 +350,7 @@
   <link name="arm_2_link">
     <inertial>
-      <mass value="0.01" />
-      <origin xyz="0 0 0" />
-      <inertia ixx="0.001" ixy="0.0" ixz="0.0" iyy="0.001" iyz="0.0" izz="0.001" />
+      <mass value="2" />
+      <origin xyz="0 0 0" />
+      <inertia ixx="0.01" ixy="0.0" ixz="0.0" iyy="0.01" iyz="0.0" izz="0.01" />
     </inertial>
     <visual>
@@ -367,12 +372,12 @@
     <parent link="arm_2_link"/>
     <child link="arm_3_link"/>
-    <limit effort="81.5" velocity="0.4189" lower="${-M_PI + safety_offset}" upper="${M_PI - safety_offset}"/>
+    <limit effort="81.5" velocity="0.4186" lower="${-M_PI + safety_offset}" upper="${M_PI - safety_offset}"/>
   </joint>
 <!-- arm_3_link -->
   <link name="arm_3_link">
     <inertial>
-      <mass value="0.01" />
-      <origin xyz="0 0 0" />
-      <inertia ixx="0.001" ixy="0.0" ixz="0.0" iyy="0.001" iyz="0.0" izz="0.001" />
+      <mass value="2" />
+      <origin xyz="0 0 0" />
+      <inertia ixx="0.01" ixy="0.0" ixz="0.0" iyy="0.01" iyz="0.0" izz="0.01" />
     </inertial>
     <visual>
@@ -394,12 +399,12 @@
     <parent link="arm_3_link"/>
     <child link="arm_4_link"/>
-    <limit effort="81.5" velocity="0.4189" lower="${-2.18 + safety_offset}" upper="${2.18 - safety_offset}"/>
+    <limit effort="81.5" velocity="0.4186" lower="${-2.18 + safety_offset}" upper="${2.18 - safety_offset}"/>
   </joint>
 <!--arm_4_link -->
   <link name="arm_4_link">
     <inertial>
-      <mass value="0.01" />
-      <origin xyz="0 0 0" />
-      <inertia ixx="0.001" ixy="0.0" ixz="0.0" iyy="0.001" iyz="0.0" izz="0.001" />
+      <mass value="2" />
+      <origin xyz="0 0 0" />
+      <inertia ixx="0.01" ixy="0.0" ixz="0.0" iyy="0.01" iyz="0.0" izz="0.01" />
     </inertial>
     <visual>
@@ -421,12 +426,12 @@
     <parent link="arm_4_link"/>
     <child link="arm_5_link"/>
-    <limit effort="20.7" velocity="0.43633" lower="${-M_PI + safety_offset}" upper="${M_PI - safety_offset}"/>
+    <limit effort="20.7" velocity="0.4363" lower="${-M_PI + safety_offset}" upper="${M_PI - safety_offset}"/>
   </joint>
 <!-- arm_5_link -->
   <link name="arm_5_link">
     <inertial>
-      <mass value="0.01" />
-      <origin xyz="0 0 0" />
-      <inertia ixx="0.001" ixy="0.0" ixz="0.0" iyy="0.001" iyz="0.0" izz="0.001" />
+      <mass value="2" />
+      <origin xyz="0 0 0" />
+      <inertia ixx="0.01" ixy="0.0" ixz="0.0" iyy="0.01" iyz="0.0" izz="0.01" />
     </inertial>
     <visual>
@@ -448,12 +453,12 @@
     <parent link="arm_5_link"/>
     <child link="arm_6_link"/>
-    <limit effort="15" velocity="1.2566" lower="${-2.09 + safety_offset}" upper="${2.09 - safety_offset}"/>
+    <limit effort="20.7" velocity="0.4363" lower="${-2.09 + safety_offset}" upper="${2.09 - safety_offset}"/>
   </joint>
 <!-- arm_6_link -->
   <link name="arm_6_link">
     <inertial>
-      <mass value="0.01" />
-      <origin xyz="0 0 0" />
-      <inertia ixx="0.001" ixy="0.0" ixz="0.0" iyy="0.001" iyz="0.0" izz="0.001" />
+      <mass value="2" />
+      <origin xyz="0 0 0" />
+      <inertia ixx="0.01" ixy="0.0" ixz="0.0" iyy="0.01" iyz="0.0" izz="0.01" />
     </inertial>
     <visual>
@@ -469,5 +474,5 @@
     </collision>
   </link>
-  <!-- joint between arm_6_link and arm_7_link -->
+<!-- joint between arm_6_link and arm_7_link -->
   <joint name="arm_7_joint" type="revolute">
     <origin xyz="0 0 0" rpy="${M_PI/2} 0 ${M_PI/2}"/>
@@ -475,12 +480,12 @@
     <parent link="arm_6_link"/>
     <child link="arm_7_link"/>
-    <limit effort="15" velocity="1.2566" lower="${-2.96 + safety_offset}" upper="${2.96 - safety_offset}"/>
+    <limit effort="4.5" velocity="0.9072" lower="${-2.96 + safety_offset}" upper="${2.96 - safety_offset}"/>
   </joint>
 <!--arm_7_link -->
   <link name="arm_7_link">
     <inertial>
-      <mass value="0.01" />
-      <origin xyz="0 0 0" />
-      <inertia ixx="0.001" ixy="0.0" ixz="0.0" iyy="0.001" iyz="0.0" izz="0.001" />
+      <mass value="2" />
+      <origin xyz="0 0 0" />
+      <inertia ixx="0.01" ixy="0.0" ixz="0.0" iyy="0.01" iyz="0.0" izz="0.01" />
     </inertial>
     <visual>
@@ -504,139 +509,9 @@
   <link name="arm_ee_link">
     <inertial>
-      <mass value="0.01" />
-      <origin xyz="0 0 0" />
-      <inertia ixx="0.001" ixy="0.0" ixz="0.0" iyy="0.001" iyz="0.0" izz="0.001" />
-    </inertial>
-  </link>
-  <!--transmission name="wheel_left_trans">
-    <type>transmission_interface/SimpleTransmission</type>
-    <joint name="wheel_left_joint">
-      <hardwareInterface>hardware_interface/VelocityJointInterface</hardwareInterface>
-    </joint>
-    <actuator name="wheel_left_motor">
-      <hardwareInterface>hardware_interface/EffortJointInterface</hardwareInterface>
-      <mechanicalReduction>0.1</mechanicalReduction>
-    </actuator>
-  </transmission>
-  <transmission name="wheel_right_trans">
-    <type>transmission_interface/SimpleTransmission</type>
-    <joint name="wheel_right_joint">
-      <hardwareInterface>hardware_interface/VelocityJointInterface</hardwareInterface>
-    </joint>
-    <actuator name="wheel_right_motor">
-      <hardwareInterface>hardware_interface/EffortJointInterface</hardwareInterface>
-      <mechanicalReduction>0.1</mechanicalReduction>
-    </actuator>
-  </transmission>
-  <transmission name="arm_1_trans">
-    <type>transmission_interface/SimpleTransmission</type>
-    <joint name="arm_1_joint">
-      <hardwareInterface>hardware_interface/PositionJointInterface</hardwareInterface>
-    </joint>
-    <actuator name="arm_1_motor">
-      <hardwareInterface>hardware_interface/EffortJointInterface</hardwareInterface>
-      <mechanicalReduction>1</mechanicalReduction>
-    </actuator>
-  </transmission>
-  <transmission name="arm_2_trans">
-    <type>transmission_interface/SimpleTransmission</type>
-    <joint name="arm_2_joint">
-      <hardwareInterface>hardware_interface/PositionJointInterface</hardwareInterface>
-    </joint>
-    <actuator name="arm_2_motor">
-      <hardwareInterface>hardware_interface/EffortJointInterface</hardwareInterface>
-      <mechanicalReduction>1</mechanicalReduction>
-    </actuator>
-  </transmission>
-  <transmission name="arm_3_trans">
-    <type>transmission_interface/SimpleTransmission</type>
-    <joint name="arm_3_joint">
-      <hardwareInterface>hardware_interface/PositionJointInterface</hardwareInterface>
-    </joint>
-    <actuator name="arm_3_motor">
-      <hardwareInterface>hardware_interface/EffortJointInterface</hardwareInterface>
-      <mechanicalReduction>1</mechanicalReduction>
-    </actuator>
-  </transmission>
-  <transmission name="arm_4_trans">
-    <type>transmission_interface/SimpleTransmission</type>
-    <joint name="arm_4_joint">
-      <hardwareInterface>hardware_interface/PositionJointInterface</hardwareInterface>
-    </joint>
-    <actuator name="arm_4_motor">
-      <hardwareInterface>hardware_interface/EffortJointInterface</hardwareInterface>
-      <mechanicalReduction>1</mechanicalReduction>
-    </actuator>
-  </transmission>
-  <transmission name="arm_5_trans">
-    <type>transmission_interface/SimpleTransmission</type>
-    <joint name="arm_5_joint">
-      <hardwareInterface>hardware_interface/PositionJointInterface</hardwareInterface>
-    </joint>
-    <actuator name="arm_5_motor">
-      <hardwareInterface>hardware_interface/EffortJointInterface</hardwareInterface>
-      <mechanicalReduction>1</mechanicalReduction>
-    </actuator>
-  </transmission>
-  <transmission name="arm_6_trans">
-    <type>transmission_interface/SimpleTransmission</type>
-    <joint name="arm_6_joint">
-      <hardwareInterface>hardware_interface/PositionJointInterface</hardwareInterface>
-    </joint>
-    <actuator name="arm_6_motor">
-      <hardwareInterface>hardware_interface/EffortJointInterface</hardwareInterface>
-      <mechanicalReduction>1</mechanicalReduction>
-    </actuator>
-  </transmission>
-  <transmission name="arm_7_trans">
-    <type>transmission_interface/SimpleTransmission</type>
-    <joint name="arm_7_joint">
-      <hardwareInterface>hardware_interface/PositionJointInterface</hardwareInterface>
-    </joint>
-    <actuator name="arm_7_motor">
-      <hardwareInterface>hardware_interface/EffortJointInterface</hardwareInterface>
-      <mechanicalReduction>1</mechanicalReduction>
-    </actuator>
-  </transmission>
-<gazebo reference="arm_base_link">
-  <gravity>true</gravity>
-  <self_collide>false</self_collide>
-  <material value="Schunk/Black"/>
-</gazebo>
-<gazebo reference="arm_1_link">
-  <gravity>true</gravity>
-  <self_collide>false</self_collide>
-  <material value="Schunk/LightGrey"/>
-</gazebo>
-<gazebo reference="arm_2_link">
-  <gravity>true</gravity>
-  <self_collide>false</self_collide>
-  <material value="Schunk/Black"/>
-</gazebo>
-<gazebo reference="arm_3_link">
-  <gravity>true</gravity>
-  <self_collide>false</self_collide>
-  <material value="Schunk/LightGrey"/>
-</gazebo>
-<gazebo reference="arm_4_link">
-  <gravity>true</gravity>
-  <self_collide>false</self_collide>
-  <material value="Schunk/Black"/>
-</gazebo>
-<gazebo reference="arm_5_link">
-  <gravity>true</gravity>
-  <self_collide>false</self_collide>
-  <material value="Schunk/LightGrey"/>
-</gazebo>
-<gazebo reference="arm_6_link">
-  <gravity>true</gravity>
-  <self_collide>false</self_collide>
-  <material value="Schunk/Black"/>
-</gazebo>
-<gazebo reference="arm_7_link">
-  <gravity>true</gravity>
-  <self_collide>false</self_collide>
-  <material value="Schunk/LightGrey"/>
-</gazebo-->
+      <mass value="1" />
+      <origin xyz="0 0 0" />
+      <inertia ixx="0.005" ixy="0.0" ixz="0.0" iyy="0.005" iyz="0.0" izz="0.005" />
+    </inertial>
+  </link>
 <gazebo>
   <plugin name="differential_drive_controller" filename="libgazebo_ros_diff_drive.so">
@@ -648,5 +523,5 @@
     <wheelSeparation>0.51</wheelSeparation>
     <wheelDiameter>0.125</wheelDiameter>
-    <torque>2.5</torque>
+    <torque>11.4</torque>  <!-- 0.95*12-->
     <commandTopic>/mp500lwa4d/mobile_base_controller/cmd_vel</commandTopic>
     <odometryTopic>odom</odometryTopic>
@@ -657,18 +532,14 @@
     <publishWheelTF>true</publishWheelTF>
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