Commit message: Add files via upload

File: mp500lwa4d_description/urdf/common.xacro (robot description, xacro)
@@ -96,5 +96,5 @@
     </joint>
     <actuator name="arm_1_motor">
-      <mechanicalReduction>596</mechanicalReduction>
+      <mechanicalReduction>1</mechanicalReduction>
     </actuator>
   </transmission>
@@ -107,5 +107,5 @@
     </joint>
     <actuator name="arm_2_motor">
-      <mechanicalReduction>596</mechanicalReduction>
+      <mechanicalReduction>1</mechanicalReduction>
     </actuator>
   </transmission>
@@ -118,5 +118,5 @@
     </joint>
     <actuator name="arm_3_motor">
-      <mechanicalReduction>625</mechanicalReduction>
+      <mechanicalReduction>1</mechanicalReduction>
     </actuator>
   </transmission>
@@ -129,5 +129,5 @@
     </joint>
     <actuator name="arm_4_motor">
-      <mechanicalReduction>625</mechanicalReduction>
+      <mechanicalReduction>1</mechanicalReduction>
     </actuator>
   </transmission>
@@ -140,5 +140,5 @@
     </joint>
     <actuator name="arm_5_motor">
-      <mechanicalReduction>552</mechanicalReduction>
+      <mechanicalReduction>1</mechanicalReduction>
     </actuator>
   </transmission>
@@ -151,5 +151,5 @@
     </joint>
     <actuator name="arm_6_motor">
-      <mechanicalReduction>552</mechanicalReduction>
+      <mechanicalReduction>1</mechanicalReduction>
     </actuator>
   </transmission>
@@ -162,5 +162,5 @@
     </joint>
     <actuator name="arm_7_motor">
-      <mechanicalReduction>300</mechanicalReduction>
+      <mechanicalReduction>1</mechanicalReduction>
     </actuator>
   </transmission>

File: mp500lwa4d_description/urdf/lwa4dmp500.urdf.xacro (robot description, xacro)
@@ -8,43 +8,4 @@
   <xacro:include filename="$(find mp500lwa4d_description)/urdf/common.xacro"/>
 <!-- Materials -->
-  <!--material name="Neobotix/Black">
-    <color rgba="0.0 0.0 0.0 1.0"/>
-  </material>
-  <material name="Neobotix/Blue">
-    <color rgba="0.0 0.0 0.8 1.0"/>
-  </material>
-  <material name="Neobotix/Green">
-    <color rgba="0.0 0.8 0.0 1.0"/>
-  </material>
-  <material name="Neobotix/Grey">
-    <color rgba="0.7 0.7 0.7 1.0"/>
-  </material>
-  <material name="Neobotix/Grey2">
-    <color rgba="0.9 0.9 0.9 1.0"/>
-  </material>
-  <material name="Neobotix/Red">
-    <color rgba="0.8 0.0 0.0 1.0"/>
-  </material>
-  <material name="Neobotix/White">
-    <color rgba="1.0 1.0 1.0 1.0"/>
-  </material>
-  <material name="Neobotix/Yellow">
-    <color rgba="1.0 1.0 0 10" />
-  </material>
-  <material name="Schunk/LightGrey">
-    <color rgba="0.7 0.7 0.7 1.0"/>
-  </material>
-  <material name="Schunk/DarkGrey">
-    <color rgba="0.4 0.4 0.4 1.0"/>
-  </material>
-  <material name="Schunk/Black">
-    <color rgba="0.0 0.0 0.0 1.0"/>
-  </material>
-  <material name="Schunk/DarkGolden">
-    <color rgba="0.4 0.4 0.3 1.0"/>
-  </material>
-  <material name="Schunk/Blue">
-    <color rgba="0.0 0.0 0.8 1.0"/>
-  </material-->
   <!--neo_mp_500-->
   <!--xacro:include filename="$(find neo_mp_500)/robot_model/mp_500/mp500.urdf.xacro" /-->
@@ -61,5 +22,5 @@
       <origin xyz="-0.160 0.0 0.09" rpy="0 0 -1.57" /><!-- for STL -->
       <geometry>
-        <mesh filename="package://neo_mp_500/robot_model/mp_500/meshes/MP500-BODY.STL" scale="0.01 0.01 0.01"/>
+        <mesh filename="package://mp500lwa4d_description/meshes/MP500-BODY.STL" scale="0.01 0.01 0.01"/>
         <!--cylinder length="0.381" radius="0.2545"/-->
         <!--box size="0.445 0.277 0.17"/-->
@@ -92,5 +53,5 @@
       <origin xyz="0 0 0" rpy="0 0 -1.57" />
       <geometry>
-	<mesh filename="package://neo_mp_500/robot_model/mp_500/meshes/MP500-WHEEL.STL" scale="0.01 0.01 0.01" />
+	<mesh filename="package://mp500lwa4d_description/meshes/MP500-WHEEL.STL" scale="0.01 0.01 0.01" />
       </geometry>
       <material name="Neobotix/Black" />
@@ -123,5 +84,5 @@
       <origin xyz="0 0 0" rpy="0 0 -1.57" />
       <geometry>
-	<mesh filename="package://neo_mp_500/robot_model/mp_500/meshes/MP500-WHEEL.STL" scale="0.01 0.01 0.01" />
+	<mesh filename="package://mp500lwa4d_description/meshes/MP500-WHEEL.STL" scale="0.01 0.01 0.01" />
       </geometry>
       <material name="Neobotix/Black"/>
@@ -161,5 +122,5 @@
       <geometry>
         <!--cylinder length="0.154" radius="0.053" /-->
-        <mesh filename="package://neo_mp_500/robot_model/mp_500/meshes/SICK-S300.STL" />
+        <mesh filename="package://mp500lwa4d_description/meshes/SICK-S300.STL" />
       </geometry>
       <material name="Neobotix/Yellow"/>
@@ -182,5 +143,5 @@
       <origin xyz="0 0 0" rpy="0 0 -1.57" />
       <geometry>
-	<mesh filename="package://neo_mp_500/robot_model/mp_500/meshes/HANGER-WHEEL.STL" scale="0.01 0.01 0.01" />
+	<mesh filename="package://mp500lwa4d_description/meshes/HANGER-WHEEL.STL" scale="0.01 0.01 0.01" />
       </geometry>
       <material name="Neobotix/Grey"/>
@@ -235,36 +196,4 @@
     <child link="castor_front" />
   </joint>
-<!--+++++++++++++++ castor_back +++++++++++++++++++++++++++-->
-  <!--link name="castor_back">
-    <inertial>
-    <mass value="0.25" />
-    <origin xyz="0 0 0" rpy="0 0 0" />
-    <inertia ixx="0.000025" ixy="0" ixz="0" iyy="0.000025" iyz="0" izz="0.000025" />
-    </inertial>
-    <visual>
-      <origin xyz="0 0 0" rpy="0 0 0" />
-      <geometry>
-        <sphere radius="0.005"/>
-      </geometry>
-      <material name="Neobotix/Grey" />
-    </visual>
-    <collision>
-      <origin xyz="0 0 0" rpy="0 0 0" />
-      <geometry>
-       <sphere radius="0.005"/>
-      </geometry>
-    </collision>
-  </link>
-  <gazebo reference="caster_back">
-   <mu1 value="0" />
-   <mu2 value="0" />
-   <kp  value="1.0" />
-   <kd  value="1.0" />
-  </gazebo-->
-  <!--joint name="castor_back_joint" type="fixed">
-    <origin xyz="-0.30 0 0.01" rpy="0 0 0"/>
-    <parent link="base_link" />
-    <child link="castor_back" />
-  </joint-->
   <!--xacro:include filename="$(find schunk_description)/urdf/common.xacro" /-->
   <!--xacro:include filename="$(find schunk_description)/urdf/materials.urdf.xacro" /-->
@@ -516,5 +445,5 @@
 <gazebo>
   <plugin name="differential_drive_controller" filename="libgazebo_ros_diff_drive.so">
-    <robotNamespace>/mp500lwa4d</robotNamespace>
+    <robotNamespace>/</robotNamespace>
     <alwaysOn>true</alwaysOn>
     <updateRate>100</updateRate>
@@ -524,8 +453,8 @@
     <wheelDiameter>0.125</wheelDiameter>
     <torque>11.4</torque>  <!-- 0.95*12-->
-    <commandTopic>/mp500lwa4d/mobile_base_controller/cmd_vel</commandTopic>
+    <commandTopic>/mobile_base_controller/cmd_vel</commandTopic>
     <odometryTopic>odom</odometryTopic>
     <odometryFrame>map</odometryFrame>
-    <robotBaseFrame>/mp500lwa4d/base_link</robotBaseFrame>
+    <robotBaseFrame>/base_link</robotBaseFrame>
     <legacyMode>false</legacyMode>
     <rosDebugLevel>Debug</rosDebugLevel>
